File: hallsensor/HallSensor.sch (KiCad schematic (older format))
At the start: 5 parts

Commit message: Misc rework.
Parts:
- removed KH1: CONN_3, symbol CONN_3
- added ANCHOR1: CONN_1, symbol CONN_1
- added PAIR1, PAIR2, PAIR3: CONN_2, symbol CONN_2
Connections:
- wire segments 20 -> 23
- no-connect marks 0 -> 1
Other:
- note added: "ANCHOR is 0.1" away from middle of sensor."
- note added: "Edge Connector"
Changed lines of the file:
@@
-EESchema Schematic File Version 2  date Monday, 07 October, 2013 01:51:57 pm
+EESchema Schematic File Version 2  date Wednesday, 09 October, 2013 02:55:02 pm
 LIBS:power
 LIBS:device
@@
 Sheet 1 1
 Title "Hall Sensor"
-Date "7 oct 2013"
+Date "9 oct 2013"
 Rev "20131007"
 Comp "ClothBot Designs"
@@
 	5000 4800 5000 5000
 Wire Wire Line
-	4800 5000 5000 5000
+	5000 5000 4800 5000
 Connection ~ 4800 5000
 Wire Wire Line
@@
 Text Notes 2000 2500 0    60   ~ 0
 - RPU* Pull-up resistors are\nunpopulated/optional.
-$Comp
-L CONN_3 KH1
-U 1 1 5252F238
-P 6350 3800
-F 0 "KH1" V 6300 3800 50  0000 C CNN
-F 1 "CONN_3" V 6400 3800 40  0000 C CNN
-F 2 "" H 6350 3800 60  0000 C CNN
-F 3 "" H 6350 3800 60  0000 C CNN
-	1    6350 3800
-	1    0    0    -1
-$EndComp
-Wire Wire Line
-	6000 3700 5600 3700
-Wire Wire Line
-	6000 3800 5600 3800
-Wire Wire Line
-	6000 3900 5600 3900
+Wire Wire Line
+	6300 3050 5900 3050
+Wire Wire Line
+	6300 3450 5900 3450
+Wire Wire Line
+	6300 3850 5900 3850
 $Comp
 L VCC #PWR08
@@
 L VCC #PWR09
 U 1 1 5252F295
-P 5600 3700
-F 0 "#PWR09" H 5600 3800 30  0001 C CNN
-F 1 "VCC" H 5600 3800 30  0000 C CNN
-F 2 "" H 5600 3700 60  0000 C CNN
-F 3 "" H 5600 3700 60  0000 C CNN
-	1    5600 3700
+P 5900 3050
+F 0 "#PWR09" H 5900 3150 30  0001 C CNN
+F 1 "VCC" H 5900 3150 30  0000 C CNN
+F 2 "" H 5900 3050 60  0000 C CNN
+F 3 "" H 5900 3050 60  0000 C CNN
+	1    5900 3050
 	1    0    0    -1
 $EndComp
@@
 L VSS #PWR010
 U 1 1 5252F29B
-P 5600 3800
-F 0 "#PWR010" H 5600 3800 30  0001 C CNN
-F 1 "VSS" H 5600 3730 30  0000 C CNN
-F 2 "" H 5600 3800 60  0000 C CNN
-F 3 "" H 5600 3800 60  0000 C CNN
-	1    5600 3800
-	1    0    0    -1
-$EndComp
-Text Label 5650 3900 0    60   ~ 0
+P 5900 3450
+F 0 "#PWR010" H 5900 3450 30  0001 C CNN
+F 1 "VSS" H 5900 3380 30  0000 C CNN
+F 2 "" H 5900 3450 60  0000 C CNN
+F 3 "" H 5900 3450 60  0000 C CNN
+	1    5900 3450
+	1    0    0    -1
+$EndComp
+Text Label 5950 3850 0    60   ~ 0
 hall1_out
+$Comp
+L CONN_1 ANCHOR1
+U 1 1 525599C0
+P 4150 5900
+F 0 "ANCHOR1" H 4230 5900 40  0000 L CNN
+F 1 "CONN_1" H 4150 5955 30  0001 C CNN
+F 2 "" H 4150 5900 60  0000 C CNN
+F 3 "" H 4150 5900 60  0000 C CNN
+	1    4150 5900
+	1    0    0    -1
+$EndComp
+NoConn ~ 4000 5900
+Text Notes 3900 6050 0    60   ~ 0
+ANCHOR is 0.1" away from middle of sensor.
+$Comp
+L CONN_2 PAIR2
+U 1 1 5255A405
+P 6650 3550
+F 0 "PAIR2" V 6600 3550 40  0000 C CNN
+F 1 "CONN_2" V 6700 3550 40  0000 C CNN
+F 2 "" H 6650 3550 60  0000 C CNN
+F 3 "" H 6650 3550 60  0000 C CNN
+	1    6650 3550
+	1    0    0    -1
+$EndComp
+$Comp
+L CONN_2 PAIR3
+U 1 1 5255A414
+P 6650 3950
+F 0 "PAIR3" V 6600 3950 40  0000 C CNN
+F 1 "CONN_2" V 6700 3950 40  0000 C CNN
+F 2 "" H 6650 3950 60  0000 C CNN
+F 3 "" H 6650 3950 60  0000 C CNN
+	1    6650 3950
+	1    0    0    -1
+$EndComp
+Wire Wire Line
+	6300 3450 6300 3650
+$Comp
+L CONN_2 PAIR1
+U 1 1 5255A3F6
+P 6650 3150
+F 0 "PAIR1" V 6600 3150 40  0000 C CNN
+F 1 "CONN_2" V 6700 3150 40  0000 C CNN
+F 2 "" H 6650 3150 60  0000 C CNN
+F 3 "" H 6650 3150 60  0000 C CNN
+	1    6650 3150
+	1    0    0    -1
+$EndComp
+Wire Wire Line
+	6300 4050 5900 4050
+$Comp
+L VCC #PWR011
+U 1 1 5255A4F7
+P 5900 4050
+F 0 "#PWR011" H 5900 4150 30  0001 C CNN
+F 1 "VCC" H 5900 4150 30  0000 C CNN
+F 2 "" H 5900 4050 60  0000 C CNN
+F 3 "" H 5900 4050 60  0000 C CNN
+	1    5900 4050
+	1    0    0    -1
+$EndComp
+Wire Wire Line
+	6300 3250 5900 3250
+Text Label 5950 3250 0    60   ~ 0
+hall1_out
+Wire Notes Line
+	6450 2950 6450 4150
+Wire Notes Line
+	6450 4150 6800 4150
+Wire Notes Line
+	6800 4150 6800 2950
+Wire Notes Line
+	6800 2950 6450 2950
+Text Notes 6450 2900 0    60   ~ 0
+Edge Connector
 $EndSCHEMATC
